File: Contra.kicad_pcb (KiCad board)
At the start: 2 copper layers, 231 x 76.2 mm, 110 parts, among them J1 Conn_01x04, SW1 SW_PUSH, U1 ProMicro

Commit message: change switch symbole and migation to kicad 7
Connections:
- D42 pad 2: Net-(D42-Pad2) -> Net-(D42-A)
- MX42 pad 2: Net-(D42-Pad2) -> Net-(D42-A)
- U1 pad 24: Net-(U1-Pad24) -> unconnected-(U1-RAW-Pad24)
Other:
- net class Default removed
- net class Power removed
