File: Contra.kicad_pcb (KiCad board)
At the start: 2 copper layers, 231 x 76.2 mm, 110 parts, among them J1 Conn_01x04, SW1 SW_PUSH, U1 ProMicro

Commit message: use smd diodes and palce on bottem select ks27 only footprint
Parts:
- removed G***: LOGO, memelogo:cartel
- removed G***: LOGO, memelogo:contra
- removed G***: LOGO, locallib:ai-ring-6mm
- removed G***: LOGO, locallib:ai-ring-6mm-FancyAss
- removed G***: LOGO, locallib:ai-ring-6mm-FancyAss-Mask
- removed J1: Conn_01x04, Pin_Headers:Pin_Header_Straight_1x04_Pitch2.54mm
- removed MX49: MX-2U, MX_Alps_Hybrid:MX-2U-ReversedStabilizers-NoLED
- D1, D10, D11, D12, D13, D14, D15, D16, D17, D18, D19, D2, D20, D21, D22, D23, D24, D25, D27, D28, D29, D3, D30, D31, D32, D33, D34, D35, D36, D37, D38, D39, D4, D40, D41, D42, D43, D44, D45, D46, D47, D48, D5, D6, D7, D8, D9: footprint locallib:D_DO-35_SOD27_P7.62mm_Horizontal-DoubleSided -> Diode_SMD:D_0805_2012Metric_Pad1.15x1.40mm_HandSolder; moved to B.Cu
- D26: value 1N4148 -> locked; footprint locallib:D_DO-35_SOD27_P7.62mm_Horizontal-DoubleSided -> Diode_SMD:D_0805_2012Metric_Pad1.15x1.40mm_HandSolder; moved to B.Cu
- MX1, MX10, MX11, MX12, MX13, MX14, MX15, MX16, MX17, MX18, MX19, MX2, MX20, MX21, MX22, MX23, MX24, MX25, MX26, MX27, MX28, MX29, MX3, MX30, MX31, MX32, MX33, MX34, MX35, MX36, MX37, MX38, MX39, MX4, MX40, MX41, MX42, MX43, MX44, MX45, MX46, MX47, MX48, MX5, MX6, MX7, MX8, MX9: footprint MX_Alps_Hybrid:MX-1U-NoLED -> WLPlanckFootprints:SW_Gateron_LowProfile_HotSwap
- moved U1 212.3 mm to (283.5, -0.51), turned to -90 degrees
- moved D3 33.7 mm to (82.3, 33.0), turned to -90 degrees
- moved D25 21.1 mm to (44.4, 72.9), turned to -90 degrees
- moved D40 17.8 mm to (101.8, 91.2), turned to -90 degrees
- moved D41 17.8 mm to (120.8, 91.2), turned to -90 degrees
- moved D38 17.5 mm to (63.4, 91.2), turned to -90 degrees
- moved D39 17.5 mm to (82.4, 91.2), turned to -90 degrees
- moved D42 17.5 mm to (139.6, 91.2), turned to -90 degrees
- moved D36 17.3 mm to (253.9, 72.9), turned to -90 degrees
- moved D12 15.1 mm to (254.0, 32.8), turned to -90 degrees
- moved D2 15.1 mm to (63.2, 32.8), turned to -90 degrees
- moved D35 13.1 mm to (234.9, 72.9), turned to -90 degrees
- moved D5 9.78 mm to (120.7, 32.5), turned to -90 degrees
- moved D1 9.76 mm to (44.5, 32.5), turned to -90 degrees
- moved D9 9.75 mm to (196.8, 32.5), turned to -90 degrees
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Connections:
- U1 pad 16: PIN15 -> unconnected-(U1-15-Pad16)
- U1 pad 17: PIN18 -> unconnected-(U1-18-Pad17)
Routing:
- net ROW1: track 249.2 -> 0.00 mm
- net COL11: track 231.4 -> 0.00 mm
- net COL10: track 212.9 -> 0.00 mm
- net COL9: track 184.7 -> 0.00 mm
- net COL8: track 164.6 -> 0.00 mm
- net COL7: track 145.4 -> 0.00 mm
- net COL6: track 127.0 -> 0.00 mm
- net COL5: track 120.6 -> 0.00 mm
- net COL0: track 109.6 -> 4.55 mm, vias 0 -> 1
- net COL4: track 93.9 -> 0.00 mm
- net GND: track 87.3 -> 1.14 mm
- net ROW0: track 268.8 -> 192.1 mm
- net +5V: track 76.2 -> 0.00 mm
- net COL1: track 73.8 -> 0.00 mm
- net COL2: track 71.4 -> 0.00 mm
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Other:
- board text removed: "Contra PCB by ai03 Revision 2.0"
- board text removed: "Pro Micro here! Component side faces away from the PCB."
